File: design_files/AST1011.brd (EAGLE design)
At the start: 10 x 10 mm, 8 parts, among them J1 SM05B, J2 SKRHABE010, U1 SX1505I087TRT

Commit message: updated documentation
Parts:
- C1: value 0.1uF -> 1uF
- J1: device tinycircuits:JST_SH_5X1 -> tinycircuits:JST_SH_5X1_EDGE
Other:
- board text added: "Wireling Joystick"
- board text removed: "Joystick Board"
Changed lines of the file:
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@@
 <layer number="59" name="Invisible" color="7" fill="1" visible="no" active="no"/>
 <layer number="61" name="stand" color="7" fill="1" visible="no" active="no"/>
+<layer number="88" name="SimResults" color="9" fill="1" visible="yes" active="yes"/>
+<layer number="89" name="SimProbes" color="9" fill="1" visible="yes" active="yes"/>
 <layer number="90" name="Modules" color="5" fill="1" visible="yes" active="yes"/>
 <layer number="91" name="Nets" color="2" fill="1" visible="no" active="no"/>
@@
 <layer number="158" name="bResistor" color="7" fill="1" visible="yes" active="yes"/>
 <layer number="159" name="henwayCAP" color="13" fill="1" visible="yes" active="yes"/>
+<layer number="160" name="IDFDebug" color="7" fill="1" visible="yes" active="yes"/>
 <layer number="191" name="mNets" color="7" fill="1" visible="no" active="no"/>
 <layer number="192" name="mBusses" color="7" fill="1" visible="no" active="no"/>
@@
 <wire x1="0" y1="40.8" x2="0" y2="0" width="0.127" layer="48"/>
 <dimension x1="15" y1="20" x2="25" y2="20" x3="20" y3="21.454653125" layer="48"/>
-<text x="38.111025" y="4.365003125" size="0.889" layer="48">Joystick Board</text>
+<text x="38.111025" y="4.365003125" size="0.889" layer="48">Wireling Joystick</text>
 <text x="34.986825" y="1.7714" size="0.889" layer="48">AS-PCB-AST1011</text>
 <text x="57.3810375" y="1.6952" size="0.889" layer="48">2</text>
@@
 <attribute name="NO_BOM" value="TRUE" x="34" y="0" size="1.778" layer="27" display="off"/>
 </element>
-<element name="J1" library="tinycircuits" package="JST_SH_5X1" value="SM05B" x="20" y="12.125">
+<element name="J1" library="tinycircuits" package="JST_SH_5X1_EDGE" value="SM05B" x="20" y="12.125">
 <attribute name="PARTNO" value="AS-ITM-00340" x="20" y="12.125" size="1.778" layer="27" display="off"/>
 <attribute name="VALUE" value="SM05B" x="20" y="12.125" size="1.778" layer="27" display="off"/>
@@
 <attribute name="VALUE" value="1.00K" x="23.1" y="16.8" size="1.778" layer="27" rot="R180" display="off"/>
 </element>
-<element name="C1" library="tinycircuits" package="C0402" value="0.1uF" x="17.1" y="15.2" rot="R270">
-<attribute name="PARTNO" value="AS-ITM-00008" x="17.1" y="15.2" size="1.778" layer="27" rot="R270" display="off"/>
-<attribute name="VALUE" value="0.1uF" x="17.1" y="15.2" size="1.778" layer="27" rot="R270" display="off"/>
+<element name="C1" library="tinycircuits" package="C0402" value="1uF" x="17.1" y="15.2" rot="R270">
+<attribute name="PARTNO" value="AS-ITM-00105" x="17.1" y="15.2" size="1.778" layer="27" rot="R270" display="off"/>
+<attribute name="VALUE" value="1uF" x="17.1" y="15.2" size="1.778" layer="27" rot="R270" display="off"/>
 </element>
 <element name="C2" library="tinycircuits" package="C0402" value="0.1uF" x="23.8" y="16" rot="R180">
@@
 <contactref element="R1" pad="1"/>
 <contactref element="U1" pad="16"/>
-<wire x1="20.2" y1="19.25" x2="20.3" y2="19.6" width="0.2032" layer="1"/>
-<wire x1="20.3" y1="19.6" x2="20.4" y2="19.7" width="0.2032" layer="1"/>
-<wire x1="20.4" y1="19.7" x2="20.7" y2="19.7" width="0.2032" layer="1"/>
-<wire x1="20.6" y1="19.25" x2="20.7" y2="19.7" width="0.2032" layer="1"/>
-<wire x1="20.7" y1="19.7" x2="22.2" y2="19.7" width="0.2032" layer="1"/>
-<wire x1="22.2" y1="19.7" x2="22.5" y2="19.4" width="0.2032" layer="1"/>
-<wire x1="22.5" y1="19.4" x2="22.5" y2="18.8" width="0.2032" layer="1"/>
-<wire x1="22.5" y1="18.8" x2="22.4" y2="18.7" width="0.2032" layer="1"/>
-<wire x1="22.4" y1="18.7" x2="22.4" y2="18.2" width="0.2032" layer="1"/>
+<wire x1="20.2" y1="19.25" x2="20.2" y2="19.6" width="0.2032" layer="1"/>
+<wire x1="20.2" y1="19.6" x2="20.6" y2="19.6" width="0.2032" layer="1"/>
+<wire x1="20.6" y1="19.25" x2="20.6" y2="19.6" width="0.2032" layer="1"/>
+<wire x1="20.6" y1="19.6" x2="22.2" y2="19.6" width="0.2032" layer="1"/>
+<wire x1="22.2" y1="19.6" x2="22.5" y2="19.3" width="0.2032" layer="1"/>
+<wire x1="22.5" y1="19.3" x2="22.5" y2="18.8" width="0.2032" layer="1"/>
+<wire x1="22.5" y1="18.8" x2="22.4" y2="18.6" width="0.2032" layer="1"/>
+<wire x1="22.4" y1="18.6" x2="22.4" y2="18.2" width="0.2032" layer="1"/>
 <wire x1="22.4" y1="18.2" x2="21.25" y2="18.2" width="0.2032" layer="1"/>
 <wire x1="19.4" y1="16.35" x2="19.4" y2="15.8" width="0.2032" layer="1"/>
@@
 <wire x1="21.25" y1="18.6" x2="21.7" y2="18.6" width="0.2032" layer="1"/>
 <wire x1="21.7" y1="18.6" x2="21.9" y2="18.8" width="0.2032" layer="1"/>
-<wire x1="21.9" y1="18.8" x2="21.9" y2="19.1" width="0.2032" layer="1"/>
-<via x="21.9" y="19.1" extent="1-16" drill="0.381"/>
-<wire x1="21.9" y1="19.1" x2="21.9" y2="18.3" width="0.2032" layer="16"/>
+<wire x1="21.9" y1="18.8" x2="21.9" y2="19" width="0.2032" layer="1"/>
+<via x="21.9" y="19" extent="1-16" drill="0.381"/>
+<wire x1="21.9" y1="19" x2="21.9" y2="18.3" width="0.2032" layer="16"/>
 <wire x1="21.9" y1="18.3" x2="21.2" y2="17.6" width="0.2032" layer="16"/>
 <wire x1="21.2" y1="17.6" x2="21.2" y2="17.3" width="0.2032" layer="16"/>
