File: design_files/AST1011.sch (EAGLE design)
At the start: 7 parts, among them J1 SM05B, J2 SKRHABE010, U1 SX1505I087TRT

Commit message: updated documentation
Parts:
- C1: value 0.1uF -> 1uF; device tinycircuits:AS-ITM-00008 -> tinycircuits:AS-ITM-00105; PARTNO (none) -> AS-ITM-00105; VALUE (none) -> 1uF
- J1: device tinycircuits:AS-ITM-00340 -> tinycircuits:AS-ITM-00340EDGE
Other:
- note added: "Joystick And I2C IO Expander"
- note added: "Variant: Standard - R"
- note added: "Wireling Joystick"
- note removed: "Joystick Board"
- note removed: "Variant: Standard"
Changed lines of the file:
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@@
 <layer number="54" name="bGND_GNDA" color="7" fill="1" visible="yes" active="no"/>
 <layer number="56" name="wert" color="7" fill="1" visible="yes" active="no"/>
-<layer number="57" name="tCAD" color="7" fill="1" visible="no" active="no"/>
-<layer number="58" name="bCAD" color="7" fill="1" visible="no" active="no"/>
-<layer number="59" name="Invisible" color="7" fill="1" visible="no" active="no"/>
-<layer number="61" name="stand" color="7" fill="1" visible="no" active="no"/>
+<layer number="57" name="tCAD" color="7" fill="1" visible="yes" active="no"/>
+<layer number="58" name="bCAD" color="7" fill="1" visible="yes" active="no"/>
+<layer number="59" name="Invisible" color="7" fill="1" visible="yes" active="no"/>
+<layer number="61" name="stand" color="7" fill="1" visible="yes" active="no"/>
+<layer number="88" name="SimResults" color="9" fill="1" visible="yes" active="yes"/>
+<layer number="89" name="SimProbes" color="9" fill="1" visible="yes" active="yes"/>
 <layer number="90" name="Modules" color="5" fill="1" visible="yes" active="yes"/>
 <layer number="91" name="Nets" color="2" fill="1" visible="yes" active="yes"/>
@@
 <layer number="158" name="bResistor" color="7" fill="1" visible="no" active="yes"/>
 <layer number="159" name="henwayCAP" color="13" fill="1" visible="yes" active="yes"/>
+<layer number="160" name="IDFDebug" color="7" fill="1" visible="yes" active="yes"/>
 <layer number="191" name="mNets" color="7" fill="1" visible="yes" active="yes"/>
 <layer number="192" name="mBusses" color="7" fill="1" visible="yes" active="yes"/>
@@
 <parts>
 <part name="FRAME1" library="tinycircuits" deviceset="FRAME_TINYCIRCUITS_B_L" device=""/>
-<part name="J1" library="tinycircuits" deviceset="AS-ITM-00340" device="" value="SM05B"/>
+<part name="J1" library="tinycircuits" deviceset="AS-ITM-00340" device="EDGE" value="SM05B"/>
 <part name="J2" library="tinycircuits" deviceset="AS-ITM-00305" device="A" value="SKRHABE010"/>
 <part name="GND5" library="tinycircuits" deviceset="GND" device=""/>
@@
 <part name="R1" library="tinycircuits" deviceset="AS-ITM-00032" device="" value="10.0K"/>
 <part name="R2" library="tinycircuits" deviceset="AS-ITM-00003" device="" value="1.00K"/>
-<part name="C1" library="tinycircuits" deviceset="AS-ITM-00008" device="" value="0.1uF"/>
+<part name="C1" library="tinycircuits" deviceset="AS-ITM-00105" device="" value="1uF">
+<attribute name="PARTNO" value="AS-ITM-00105"/>
+<attribute name="VALUE" value="1uF"/>
+</part>
 <part name="GND2" library="tinycircuits" deviceset="GND" device=""/>
 <part name="P+4" library="tinycircuits" deviceset="VCC" device=""/>
@@
 <sheet>
 <plain>
-<text x="340.868" y="17.272" size="3.556" layer="94" font="vector">Joystick Board</text>
+<text x="340.868" y="17.272" size="3.556" layer="94" font="vector">Wireling Joystick</text>
 <text x="327.152" y="6.35" size="3.556" layer="94" font="vector">AS-SCH-AST1011</text>
 <text x="416.56" y="6.858" size="3.556" layer="94" font="vector">2</text>
-<text x="182.88" y="187.96" size="5.08" layer="94" font="vector">Joystick Board</text>
+<text x="129.54" y="177.8" size="5.08" layer="94" font="vector">Joystick And I2C IO Expander</text>
 <text x="45.72" y="35.56" size="3.048" layer="91">Released under the Creative Commons Attribution Share-Alike 3.0 License</text>
 <text x="45.72" y="30.48" size="3.048" layer="91">http://creativecommons.org/licenses/by-sa/3.0</text>
@@
 <text x="50.8" y="50.8" size="1.778" layer="96">Hand Populated: -</text>
 <text x="50.8" y="48.26" size="1.778" layer="96">Hand Soldered: -</text>
-<text x="50.8" y="55.88" size="1.778" layer="96">Variant: Standard</text>
+<text x="50.8" y="55.88" size="1.778" layer="96">Variant: Standard - R</text>
 <text x="50.8" y="45.72" size="1.778" layer="96">Notes: -</text>
 </plain>
